Commit message: setup yml and sphere for b1_z1

File: src/culoco/content/assets/robot/B1_Z1/urdf/b1.urdf (robot description, URDF)
Before this commit: robot b1_description, 45 links, 44 joints
Links:
- added link arm_ee_link
Joints:
- added joint ee_fixed_joint: type fixed, parent gripperMover, child arm_ee_link, origin xyz=0.085 0 -0.017 rpy=0 0 0
